Commit message: controller

File: src/kuka_description/urdf/kuka_iiwa.xacro (robot description, xacro)
@@ -97,8 +97,8 @@
       link="link1" />
     <axis
-      xyz="0 0 -1" />
-    <limit
-      lower="-2.97"
-      upper="2.97"
+      xyz="0 0 1" />
+    <limit
+      lower="-3.141"
+      upper="3.141"
       effort="176"
       velocity="1.71" />
@@ -157,6 +157,6 @@
       xyz="0 0 1" />
     <limit
-      lower="-2.09"
-      upper="2.09"
+      lower="-3.141"
+      upper="3.141"
       effort="176"
       velocity="1.71" />
@@ -213,8 +213,8 @@
       link="link3" />
     <axis
-      xyz="0 0 -1" />
-    <limit
-      lower="-2.97"
-      upper="2.97"
+      xyz="0 0 1" />
+    <limit
+      lower="-3.141"
+      upper="3.141"
       effort="110"
       velocity="1.75" />
@@ -271,8 +271,8 @@
       link="link4" />
     <axis
-      xyz="0 0 -1" />
-    <limit
-      lower="-2.09"
-      upper="2.09"
+      xyz="0 0 1" />
+    <limit
+      lower="-3.141"
+      upper="3.141"
       effort="110"
       velocity="2.27" />
@@ -329,8 +329,8 @@
       link="link5" />
     <axis
-      xyz="0 0 -1" />
-    <limit
-      lower="-2.97"
-      upper="2.97"
+      xyz="0 0 1" />
+    <limit
+      lower="-3.141"
+      upper="3.141"
       effort="110"
       velocity="2.44" />
@@ -389,6 +389,6 @@
       xyz="0 0 1" />
     <limit
-      lower="-2.09"
-      upper="2.09"
+      lower="-3.141"
+      upper="3.141"
       effort="40"
       velocity="3.14" />
@@ -447,6 +447,6 @@
       xyz="0 0 1" />
     <limit
-      lower="-3.05"
-      upper="3.05"
+      lower="-3.141"
+      upper="3.141"
       effort="40"
       velocity="3.14" />
